File: CoffeeMonitor V1.kicad_pcb (KiCad board)
At the start: 2 copper layers, 1 part, among them U1 ESP32-S3-WROOM-2

Commit message: Finished CoffeeMonitor PCB
Parts:
- added C1: 4.7uF, Capacitor_SMD:C_1206_3216Metric, F.Cu at (138.6, 86.9)
- added C10: 10uF, Capacitor_SMD:C_0603_1608Metric, F.Cu at (237.9, 96.2)
- added C11: 100nF, Capacitor_SMD:C_0402_1005Metric, F.Cu at (240.1, 106.7)
- added C12: 100nF, Capacitor_SMD:C_0402_1005Metric, F.Cu at (237.9, 94.7)
- added C13: 10uF, Capacitor_SMD:C_0603_1608Metric, F.Cu at (239.5, 57.0)
- added C14: 100nF, Capacitor_SMD:C_0402_1005Metric, F.Cu at (240.0, 58.5)
- added C16: 10uF, Capacitor_SMD:C_0603_1608Metric, F.Cu at (148.8, 73.2)
- added C17: 100nF, Capacitor_SMD:C_0402_1005Metric, F.Cu at (147.2, 73.8)
- added C18: 10uF, Capacitor_SMD:C_0603_1608Metric, F.Cu at (236.1, 57.8)
- added C2: 4.7uF, Capacitor_SMD:C_1206_3216Metric, F.Cu at (151.1, 86.9)
- added C3: 4.7uF, Capacitor_SMD:C_1206_3216Metric, F.Cu at (163.1, 86.9)
- added C4: 4.7uF, Capacitor_SMD:C_1206_3216Metric, F.Cu at (175.6, 86.9)
- added C5: 10uF, Capacitor_SMD:C_0603_1608Metric, F.Cu at (233.7, 50.0)
- added C6: 10uF, Capacitor_SMD:C_0603_1608Metric, F.Cu at (220.9, 42.4)
- added C7: JVJ10V100M5X5, ELECTROLITIC CAPACITORS:CAP-SMD_BD5.0-L5.3-W5.3-LS6.0-FD-H5.7, F.Cu at (237.0, 115.2)
- added C8: 10uF, Capacitor_SMD:C_0603_1608Metric, F.Cu at (205.0, 51.4)
- added C9: 10uF, Capacitor_SMD:C_0603_1608Metric, F.Cu at (239.6, 108.1)
- added F1: MF2410F1.000TM, FUSES:F2410, F.Cu at (186.0, 103.5)
- added H1: MountingHole, MountingHole:MountingHole_3.2mm_M3, F.Cu at (245.2, 40.0)
- added H2: MountingHole, MountingHole:MountingHole_3.2mm_M3, F.Cu at (245.2, 52.0)
- added H3: MountingHole, MountingHole:MountingHole_3.2mm_M3, F.Cu at (148.5, 80.8)
- added H4: MountingHole, MountingHole:MountingHole_3.2mm_M3, F.Cu at (184.0, 87.0)
- added H5: 2.54-1*4P母, CONNECTORS:HDR-TH_4P-P2.54-V-F, F.Cu at (239.7, 86.1)
- added L1: 47nH, Inductor_SMD:L_0402_1005Metric, F.Cu at (227.9, 40.0)
- added LED1: ORH-B36G, LEDS:LED0603-RD, F.Cu at (219.6, 50.8)
- added LED2: 0805G (Green), LEDS:LED0805-R-RD, F.Cu at (142.3, 52.7)
- added LED3: 0805G (Green), LEDS:LED0805-R-RD, F.Cu at (155.1, 52.6)
- added LED4: 0805G (Green), LEDS:LED0805-R-RD, F.Cu at (167.0, 52.5)
- added LED5: 0805G (Green), LEDS:LED0805-R-RD, F.Cu at (179.5, 52.5)
- added LED6: 0805G (Green), LEDS:LED0805-R-RD, F.Cu at (237.8, 110.2)
- added P1: WJ500V-5.08-2P-14-00A, CONNECTORS:CONN-TH_2P-P5.00_WJ500V-5.08-2P, F.Cu at (136.6, 113.9)
- added P2: WJ500V-5.08-2P-14-00A, CONNECTORS:CONN-TH_2P-P5.00_WJ500V-5.08-2P, F.Cu at (149.1, 113.8)
- added P3: WJ500V-5.08-2P-14-00A, CONNECTORS:CONN-TH_2P-P5.00_WJ500V-5.08-2P, F.Cu at (161.2, 113.9)
- added P4: WJ500V-5.08-2P-14-00A, CONNECTORS:CONN-TH_2P-P5.00_WJ500V-5.08-2P, F.Cu at (173.7, 113.8)
- added P5: WJ500V-5.08-2P-14-00A, CONNECTORS:CONN-TH_2P-P5.00_WJ500V-5.08-2P, F.Cu at (137.0, 43.4)
- added P6: WJ500V-5.08-2P-14-00A, CONNECTORS:CONN-TH_2P-P5.00_WJ500V-5.08-2P, F.Cu at (149.6, 43.4)
- added P7: WJ500V-5.08-2P-14-00A, CONNECTORS:CONN-TH_2P-P5.00_WJ500V-5.08-2P, F.Cu at (161.6, 43.4)
- added P8: WJ500V-5.08-2P-14-00A, CONNECTORS:CONN-TH_2P-P5.00_WJ500V-5.08-2P, F.Cu at (174.1, 43.4)
- added P9: WJ500V-5.08-2P-14-00A, CONNECTORS:CONN-TH_2P-P5.00_WJ500V-5.08-2P, F.Cu at (186.0, 113.8)
- added PJ1: PJ-307_C2939173, CONNECTORS:AUDIO-TH_PJ-307, F.Cu at (200.5, 45.2)
- added PJ2: PJ-307_C2939173, CONNECTORS:AUDIO-TH_PJ-307, F.Cu at (188.0, 45.2)
- added PS1: HLK-5M05, Converter_ACDC:Converter_ACDC_Hi-Link_HLK-5Mxx, F.Cu at (196.5, 103.5)
- added R1: 68k, Resistor_SMD:R_2512_6332Metric, F.Cu at (134.1, 104.4)
- added R10: 10k, Resistor_SMD:R_0402_1005Metric, F.Cu at (138.0, 61.7)
- added R11: 2.2k, Resistor_SMD:R_0603_1608Metric, F.Cu at (150.5, 49.4)
- added R12: 10k, Resistor_SMD:R_0402_1005Metric, F.Cu at (150.5, 61.7)
- added R13: 2.2k, Resistor_SMD:R_0603_1608Metric, F.Cu at (162.7, 49.4)
- added R14: 10k, Resistor_SMD:R_0402_1005Metric, F.Cu at (162.5, 61.7)
- added R15: 2.2k, Resistor_SMD:R_0603_1608Metric, F.Cu at (175.1, 49.4)
- added R16: 10k, Resistor_SMD:R_0402_1005Metric, F.Cu at (175.2, 61.5)
- added R17: 680, Resistor_SMD:R_0402_1005Metric, F.Cu at (220.3, 49.0)
- added R18: 10k, Resistor_SMD:R_0402_1005Metric, F.Cu at (140.5, 51.7)
- added R19: 10k, Resistor_SMD:R_0402_1005Metric, F.Cu at (153.3, 51.7)
- added R2: 68k, Resistor_SMD:R_2512_6332Metric, F.Cu at (146.6, 104.3)
- added R20: 10k, Resistor_SMD:R_0402_1005Metric, F.Cu at (165.3, 51.4)
- added R21: 10k, Resistor_SMD:R_0402_1005Metric, F.Cu at (177.8, 51.4)
- added R22: 10k, Resistor_SMD:R_0402_1005Metric, F.Cu at (227.8, 53.5)
- added R23: 10k, Resistor_SMD:R_0402_1005Metric, F.Cu at (205.5, 52.9)
- added R24: 10k, Resistor_SMD:R_0402_1005Metric, F.Cu at (203.5, 52.9)
- added R25: 10k, Resistor_SMD:R_0402_1005Metric, F.Cu at (192.5, 51.4)
- added R26: 10k, Resistor_SMD:R_0402_1005Metric, F.Cu at (223.8, 39.6)
- added R27: 10k, Resistor_SMD:R_0402_1005Metric, F.Cu at (225.3, 39.6)
- added R28: 1k, Resistor_SMD:R_0402_1005Metric, F.Cu at (234.8, 110.2)
- added R29: 5.1k, Resistor_SMD:R_0402_1005Metric, F.Cu at (237.9, 58.5)
- added R3: 68k, Resistor_SMD:R_2512_6332Metric, F.Cu at (158.6, 103.9)
- added R30: 10k, Resistor_SMD:R_0402_1005Metric, F.Cu at (146.8, 76.5)
- added R31: 33, Resistor_SMD:R_0402_1005Metric, F.Cu at (220.4, 73.6)
- added R32: 10k, Resistor_SMD:R_0402_1005Metric, F.Cu at (146.6, 67.8)
- added R33: 33, Resistor_SMD:R_0402_1005Metric, F.Cu at (220.4, 72.4)
- added R34: 33, Resistor_SMD:R_0402_1005Metric, F.Cu at (147.1, 70.6)
- added R35: 10k, Resistor_SMD:R_0402_1005Metric, F.Cu at (235.8, 79.8)
- added R36: 10k, Resistor_SMD:R_0402_1005Metric, F.Cu at (147.0, 69.5)
- added R37: 10k, Resistor_SMD:R_0402_1005Metric, F.Cu at (150.2, 73.8)
- added R4: 68k, Resistor_SMD:R_2512_6332Metric, F.Cu at (171.1, 103.8)
- added R5: 10k, Resistor_SMD:R_0805_2012Metric, F.Cu at (134.2, 86.9)
- added R6: 10k, Resistor_SMD:R_0805_2012Metric, F.Cu at (146.6, 86.9)
- added R7: 10k, Resistor_SMD:R_0805_2012Metric, F.Cu at (158.5, 86.9)
- added R8: 10k, Resistor_SMD:R_0805_2012Metric, F.Cu at (171.2, 86.9)
- added R9: 2.2k, Resistor_SMD:R_0603_1608Metric, F.Cu at (138.0, 49.4)
- added SW1: ENABLE, BUTTONS:SW-SMD_4P-L5.1-W5.1-P3.70-LS6.5-TL_H1.5, F.Cu at (238.6, 52.0)
- added SW2: BOOT, BUTTONS:SW-SMD_4P-L5.1-W5.1-P3.70-LS6.5-TL_H1.5, F.Cu at (234.0, 88.1)
- added TF1: SH-TF-01A, CONNECTORS:TF-SMD_SH_SH-TF-01A, F.Cu at (139.7, 74.9)
- added U10: ATGM336H-5N31, GPS:GPSM-SMD_ATGM336H-TR, F.Cu at (227.3, 46.7)
- added U11: AT24C32M/TR, EEPROM:SOP-8_L4.9-W3.9-P1.27-LS6.0-BL, F.Cu at (216.2, 43.4)
- added U12: BWU.FL-IPEX1, CONNECTORS:IPEX-SMD_BWIPX-1-001E, F.Cu at (230.6, 38.7)
- added U14: AMS1117-3.3, Package_TO_SOT_SMD:SOT-223-3_TabPin2, F.Cu at (237.9, 101.6)
- added U2: PC817, Package_DIP:DIP-4_W7.62mm, F.Cu at (150.6, 51.6)
- added U3: PC817, Package_DIP:DIP-4_W7.62mm, F.Cu at (162.6, 51.6)
- added U4: PC817, Package_DIP:DIP-4_W7.62mm, F.Cu at (175.1, 51.6)
- added U5: H11AA1M, OPTOISOLATORS:PDIP-6_L8.5-W6.5-P2.54-LS7.6-BL, F.Cu at (136.6, 93.9)
- added U6: H11AA1M, OPTOISOLATORS:PDIP-6_L8.5-W6.5-P2.54-LS7.6-BL, F.Cu at (149.1, 93.8)
- added U7: H11AA1M, OPTOISOLATORS:PDIP-6_L8.5-W6.5-P2.54-LS7.6-BL, F.Cu at (161.1, 93.9)
- added U8: H11AA1M, OPTOISOLATORS:PDIP-6_L8.5-W6.5-P2.54-LS7.6-BL, F.Cu at (173.6, 93.8)
- added U9: ESP32-S3-WROOM-1(N16R8), MCUs:WIRELM-SMD_ESP32-S3-WROOM-1, F.Cu at (231.3, 69.2)
- U1: value ESP32-S3-WROOM-2 -> PC817; footprint RF_Module:ESP32-S3-WROOM-2 -> Package_DIP:DIP-4_W7.62mm
- moved U1 87.5 mm to (138.0, 51.6), turned to -90 degrees
Connections:
- U1 pad 1: Net-(U1-GND-Pad1) -> Net-(R9-Pad2)
- U1 pad 2: unconnected-(U1-3V3-Pad2) -> Net-(LED2-K)
- U1 pad 3: unconnected-(U1-EN-Pad3) -> GND
- U1 pad 4: unconnected-(U1-IO4-Pad4) -> /IO14
Routing:
- net /IO41: track 0.00 -> 107.0 mm, vias 0 -> 2
- net /IO42: track 0.00 -> 95.7 mm, vias 0 -> 2
- net /IO14: track 0.00 -> 89.5 mm
- net /IO2: track 0.00 -> 86.5 mm, vias 0 -> 2
- net /CARD_DETECT: track 0.00 -> 79.6 mm
- net /CS: track 0.00 -> 78.0 mm
- net Net-(TF1-CLK): track 0.00 -> 77.2 mm
- net /IO13: track 0.00 -> 76.5 mm
- net /MISO: track 0.00 -> 76.2 mm
- net Net-(TF1-CMD): track 0.00 -> 76.2 mm
- net /IO1: track 0.00 -> 74.8 mm, vias 0 -> 2
- net /IO12: track 0.00 -> 63.8 mm
- net +3.3V: track 0.00 -> 59.7 mm, vias 0 -> 23
- net /IO11: track 0.00 -> 50.7 mm
- net /ADC1_CH7: track 0.00 -> 39.0 mm
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- added copper zone on In2.Cu, net +3.3V
- added copper zone on In2.Cu, net +5V
- added copper zone on F.Cu, net GND
Other:
- board outline added: 119.2 x 85 mm
- copper layers 2 -> 4
- board text added: "+"
- board text added: "-"
- board text added: "BOOT"
- board text added: "CoffeeMonitor v2.0 11/11/25"
- board text added: "GPS"
- board text added: "HIGH VOLTAGE"
- board text added: "POWER"
- board text added: "RESET"
- board text added: "RX"
- board text added: "TEMP"
- board text added: "TX"
